File: contender.sch (KiCad schematic (older format))
At the start: 77 parts

Commit message: fixup scheme
Parts:
- removed D? (x24): SOD-123, Diodes_SMD:D_SOD-123, symbol Device:D_Small
- removed D? (x4): WS2812B, LEDs:LED_WS2812B-PLCC4, symbol LED:WS2812B
- removed MX-E-? (x2), MX?: MX-2U, MX_Alps_Hybrid:MX-2U-ReversedStabilizers, symbol MX_Alps_Hybrid:MX-NoLED
- removed MX? (x24): MX-1U, MX_Alps_Hybrid:MX-1U, symbol MX_Alps_Hybrid:MX-NoLED
- added CR10, CR11, CR12, CR13, CR14, CR15, CR16, CR17, CR18, CR19, CR20, CR21, CR22, CR23, CR24, CR25, CR26, CR27, CR28, CR29, CR30, CR31, CR32, CR33, CR34, CR35, CR36, CR37, CR38, CR5, CR6, CR7, CR8, CR9: 0.1u, Capacitor_SMD:C_0603_1608Metric, symbol Device:C_Small
- added D1, D10, D11, D12, D13, D14, D15, D16, D17, D18, D19, D2, D20, D21, D22, D23, D24, D25, D26, D27, D3, D4, D5, D6, D7, D8, D9: 1N4148W, Diode_SMD:D_SOD-123, symbol Diode:1N4148W
- added L1, L10, L11, L12, L13, L14, L15, L16, L17, L18, L19, L2, L20, L21, L22, L23, L24, L25, L26, L27, L28, L29, L3, L30, L31, L32, L33, L34, L4, L5, L6, L7, L8, L9: YS-SK6812MINI-E, sk6812mini-e:YS-SK6812_backlight, symbol YS-SK6812MINI-E:YS-SK6812MINI-E
- added L35, L36, L37, L38: YS-SK6812MINI-E, sk6812mini-e:YS-SK6812_underglow, symbol YS-SK6812MINI-E:YS-SK6812MINI-E
- added MX-E-1, MX-E-2, MX-E-3: MX-2U, MX_Only:MXOnly-2U-Hotswap-ReversedStabilizers, symbol MX_Alps_Hybrid:MX-NoLED
- added MX1, MX10, MX11, MX12, MX13, MX14, MX15, MX16, MX17, MX18, MX19, MX2, MX20, MX21, MX22, MX23, MX24, MX25, MX26, MX27, MX3, MX4, MX5, MX6, MX7, MX8, MX9: MX-1U, MX_Only:MXOnly-1U-Hotswap, symbol MX_Alps_Hybrid:MX-NoLED
- C1, C2, C3, C4, C5, C6: renamed from C?; footprint Capacitors_SMD:C_0603 -> Capacitor_SMD:C_0603_1608Metric
- CR1, CR2, CR3, CR4: renamed from CR?; footprint Capacitors_SMD:C_0603 -> Capacitor_SMD:C_0603_1608Metric
- F1: renamed from F?; footprint Fuse_Holders_and_Fuses:Fuse_SMD1206_Reflow -> Fuse:Fuse_1206_3216Metric
- R1, R2, R3, R4, R5, R6: renamed from R?; footprint Resistors_SMD:R_0805 -> Resistor_SMD:R_0805_2012Metric
- U1: renamed from U?; footprint Housings_DFN_QFN:QFN-32-1EP_5x5mm_Pitch0.5mm -> keyboard_parts:QFN-32-1EP_5x5mm_Pitch0.5mm
- USB1: renamed from USB?; footprint (none) -> Type-C:HRO-TYPE-C-31-M-12-Assembly
- Y1: renamed from Y?; footprint Crystals:Crystal_SMD_3225-4pin_3.2x2.5mm -> Crystal:Crystal_SMD_3225-4Pin_3.2x2.5mm
- gave numbers to parts that had none: 2
Connections:
- net labels added: COL4
- wire segments 172 -> 544
Other:
- moved on the sheet: C1, C2, C3, C4, C5, C6, CR1, CR2, CR3, CR4, R1, R6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

Commit message: 1.0 finish up
Parts:
- removed CR34, CR35, CR36, CR37, CR38: 0.1u, Capacitor_SMD:C_0603_1608Metric, symbol Device:C_Small
- removed D24: 1N4148W, Diode_SMD:D_SOD-123, symbol Diode:1N4148W
- removed L34: YS-SK6812MINI-E, sk6812mini-e:YS-SK6812_backlight, symbol YS-SK6812MINI-E:YS-SK6812MINI-E
- removed L35, L36, L37, L38: YS-SK6812MINI-E, sk6812mini-e:YS-SK6812_underglow, symbol YS-SK6812MINI-E:YS-SK6812MINI-E
- removed MX-E-1, MX-E-2, MX-E-3: MX-2U, MX_Only:MXOnly-2U-Hotswap-ReversedStabilizers, symbol MX_Alps_Hybrid:MX-NoLED
- removed MX24: MX-1U, MX_Only:MXOnly-1U-Hotswap, symbol MX_Alps_Hybrid:MX-NoLED
- MX20: value MX-1U -> MX-2U; footprint MX_Only:MXOnly-1U-Hotswap -> MX_Only:MXOnly-2U-Hotswap-ReversedStabilizers
- renumbered D25 to D24, D26 to D25, D27 to D26, MX25 to MX24, MX26 to MX25, MX27 to MX26
Connections:
- net +5V: now also L29.1 (VDD), L30.1 (VDD)
- net COL0: now also U1.22 (PC7); no longer U1.10 (PD4)
- net COL1: now also U1.12 (PD6); no longer U1.11 (PD5)
- net COL3: now also U1.14 (PB0); no longer U1.16 (PB2)
- net COL4: now also U1.15 (PB1); no longer U1.19 (PB5)
- net RGBLED: now also U1.23 (PC6)
- net ROW0: now also U1.9 (PD3); no longer U1.26 (PC4)
- net ROW1: now also U1.19 (PB5); no longer U1.25 (PC5)
- net ROW2: now also U1.21 (PB7); no longer U1.12 (PD6)
- net ROW3: now also U1.18 (PB4); no longer U1.13 (~HWB~/PD7)
- net ROW4: now also U1.16 (PB2); no longer U1.20 (PB6)
- net ROWFN: now also U1.10 (PD4); no longer U1.23 (PC6)
- net at R6.2: now also U1.13 (~HWB~/PD7); no longer U1.7 (PD1)
- no-connect marks 3 -> 11
Other:
- note added: "1.0"
- note added: "2020-10-29"
- note added: "Contender"
- moved on the sheet: L33, R6

Commit message: fix led footpring & v1.1 commit
Parts:
- L1, L10, L11, L12, L13, L14, L15, L16, L17, L18, L19, L2, L20, L21, L22, L23, L24, L25, L26, L27, L28, L29, L3, L30, L31, L32, L33, L4, L5, L6, L7, L8, L9: footprint sk6812mini-e:YS-SK6812_backlight -> sk6812mini-e:YS-SK6812-MINI-E_backlight
- U1: value ATmega32U2-AU -> ATmega32U2-MU; symbol MCU_Microchip_ATmega:ATmega32U2-AU -> MCU_Microchip_ATmega:ATmega32U2-MU
Connections:
- net GND: now also U1.33 (GND)
Other:
- note added: "1.1"
- note removed: "1.0"
Changed lines of the file:
@@
 Connection ~ 2200 4000
 $Comp
-L MCU_Microchip_ATmega:ATmega32U2-AU U1
+L MCU_Microchip_ATmega:ATmega32U2-MU U1
 U 1 1 5F759979
 P 2300 2600
 F 0 "U1" H 2300 1114 50  0000 C CNN
-F 1 "ATmega32U2-AU" H 2300 1023 50  0000 C CNN
+F 1 "ATmega32U2-MU" H 2300 1023 50  0000 C CNN
 F 2 "keyboard_parts:QFN-32-1EP_5x5mm_Pitch0.5mm" H 2300 2600 50  0001 C CIN
 F 3 "http://ww1.microchip.com/downloads/en/DeviceDoc/doc7799.pdf" H 2300 2600 50  0001 C CNN
@@
 F 0 "L1" H 5050 1038 51  0000 C CNN
 F 1 "YS-SK6812MINI-E" H 5050 1103 16  0000 C CNN
-F 2 "sk6812mini-e:YS-SK6812_backlight" H 5050 1300 60  0001 C CNN
+F 2 "sk6812mini-e:YS-SK6812-MINI-E_backlight" H 5050 1300 60  0001 C CNN
 F 3 "" H 5050 1300 60  0001 C CNN
 	1    5050 1300
@@
 F 0 "L2" H 5650 1038 51  0000 C CNN
 F 1 "YS-SK6812MINI-E" H 5650 1103 16  0000 C CNN
-F 2 "sk6812mini-e:YS-SK6812_backlight" H 5650 1300 60  0001 C CNN
+F 2 "sk6812mini-e:YS-SK6812-MINI-E_backlight" H 5650 1300 60  0001 C CNN
 F 3 "" H 5650 1300 60  0001 C CNN
 	1    5650 1300
@@
 F 0 "L3" H 6250 1038 51  0000 C CNN
 F 1 "YS-SK6812MINI-E" H 6250 1103 16  0000 C CNN
-F 2 "sk6812mini-e:YS-SK6812_backlight" H 6250 1300 60  0001 C CNN
+F 2 "sk6812mini-e:YS-SK6812-MINI-E_backlight" H 6250 1300 60  0001 C CNN
 F 3 "" H 6250 1300 60  0001 C CNN
 	1    6250 1300
@@
 F 0 "L4" H 6850 1038 51  0000 C CNN
 F 1 "YS-SK6812MINI-E" H 6850 1103 16  0000 C CNN
-F 2 "sk6812mini-e:YS-SK6812_backlight" H 6850 1300 60  0001 C CNN
+F 2 "sk6812mini-e:YS-SK6812-MINI-E_backlight" H 6850 1300 60  0001 C CNN
 F 3 "" H 6850 1300 60  0001 C CNN
 	1    6850 1300
@@
 F 0 "L8" H 6850 1538 51  0000 C CNN
 F 1 "YS-SK6812MINI-E" H 6850 1603 16  0000 C CNN
-F 2 "sk6812mini-e:YS-SK6812_backlight" H 6850 1800 60  0001 C CNN
+F 2 "sk6812mini-e:YS-SK6812-MINI-E_backlight" H 6850 1800 60  0001 C CNN
 F 3 "" H 6850 1800 60  0001 C CNN
 	1    6850 1800
@@
 F 0 "L7" H 6250 1538 51  0000 C CNN
 F 1 "YS-SK6812MINI-E" H 6250 1603 16  0000 C CNN
-F 2 "sk6812mini-e:YS-SK6812_backlight" H 6250 1800 60  0001 C CNN
+F 2 "sk6812mini-e:YS-SK6812-MINI-E_backlight" H 6250 1800 60  0001 C CNN
 F 3 "" H 6250 1800 60  0001 C CNN
 	1    6250 1800
@@
 F 0 "L6" H 5650 1538 51  0000 C CNN
 F 1 "YS-SK6812MINI-E" H 5650 1603 16  0000 C CNN
-F 2 "sk6812mini-e:YS-SK6812_backlight" H 5650 1800 60  0001 C CNN
+F 2 "sk6812mini-e:YS-SK6812-MINI-E_backlight" H 5650 1800 60  0001 C CNN
 F 3 "" H 5650 1800 60  0001 C CNN
 	1    5650 1800
@@
 F 0 "L5" H 5050 1538 51  0000 C CNN
 F 1 "YS-SK6812MINI-E" H 5050 1603 16  0000 C CNN
-F 2 "sk6812mini-e:YS-SK6812_backlight" H 5050 1800 60  0001 C CNN
+F 2 "sk6812mini-e:YS-SK6812-MINI-E_backlight" H 5050 1800 60  0001 C CNN
 F 3 "" H 5050 1800 60  0001 C CNN
 	1    5050 1800
@@
 F 0 "L12" H 6850 2038 51  0000 C CNN
 F 1 "YS-SK6812MINI-E" H 6850 2103 16  0000 C CNN
-F 2 "sk6812mini-e:YS-SK6812_backlight" H 6850 2300 60  0001 C CNN
+F 2 "sk6812mini-e:YS-SK6812-MINI-E_backlight" H 6850 2300 60  0001 C CNN
 F 3 "" H 6850 2300 60  0001 C CNN
 	1    6850 2300
@@
 F 0 "L11" H 6250 2038 51  0000 C CNN
 F 1 "YS-SK6812MINI-E" H 6250 2103 16  0000 C CNN
-F 2 "sk6812mini-e:YS-SK6812_backlight" H 6250 2300 60  0001 C CNN
+F 2 "sk6812mini-e:YS-SK6812-MINI-E_backlight" H 6250 2300 60  0001 C CNN
 F 3 "" H 6250 2300 60  0001 C CNN
 	1    6250 2300
@@
 F 0 "L10" H 5650 2038 51  0000 C CNN
 F 1 "YS-SK6812MINI-E" H 5650 2103 16  0000 C CNN
-F 2 "sk6812mini-e:YS-SK6812_backlight" H 5650 2300 60  0001 C CNN
+F 2 "sk6812mini-e:YS-SK6812-MINI-E_backlight" H 5650 2300 60  0001 C CNN
 F 3 "" H 5650 2300 60  0001 C CNN
 	1    5650 2300
@@
 F 0 "L9" H 5050 2038 51  0000 C CNN
 F 1 "YS-SK6812MINI-E" H 5050 2103 16  0000 C CNN
-F 2 "sk6812mini-e:YS-SK6812_backlight" H 5050 2300 60  0001 C CNN
+F 2 "sk6812mini-e:YS-SK6812-MINI-E_backlight" H 5050 2300 60  0001 C CNN
 F 3 "" H 5050 2300 60  0001 C CNN
 	1    5050 2300
@@
 F 0 "L16" H 6850 2538 51  0000 C CNN
 F 1 "YS-SK6812MINI-E" H 6850 2603 16  0000 C CNN
-F 2 "sk6812mini-e:YS-SK6812_backlight" H 6850 2800 60  0001 C CNN
+F 2 "sk6812mini-e:YS-SK6812-MINI-E_backlight" H 6850 2800 60  0001 C CNN
 F 3 "" H 6850 2800 60  0001 C CNN
 	1    6850 2800
@@
 F 0 "L13" H 5050 2538 51  0000 C CNN
 F 1 "YS-SK6812MINI-E" H 5050 2603 16  0000 C CNN
-F 2 "sk6812mini-e:YS-SK6812_backlight" H 5050 2800 60  0001 C CNN
+F 2 "sk6812mini-e:YS-SK6812-MINI-E_backlight" H 5050 2800 60  0001 C CNN
 F 3 "" H 5050 2800 60  0001 C CNN
 	1    5050 2800
@@
 F 0 "L14" H 5650 2538 51  0000 C CNN
 F 1 "YS-SK6812MINI-E" H 5650 2603 16  0000 C CNN
-F 2 "sk6812mini-e:YS-SK6812_backlight" H 5650 2800 60  0001 C CNN
+F 2 "sk6812mini-e:YS-SK6812-MINI-E_backlight" H 5650 2800 60  0001 C CNN
 F 3 "" H 5650 2800 60  0001 C CNN
 	1    5650 2800
@@
 F 0 "L15" H 6250 2538 51  0000 C CNN
 F 1 "YS-SK6812MINI-E" H 6250 2603 16  0000 C CNN
-F 2 "sk6812mini-e:YS-SK6812_backlight" H 6250 2800 60  0001 C CNN
+F 2 "sk6812mini-e:YS-SK6812-MINI-E_backlight" H 6250 2800 60  0001 C CNN
 F 3 "" H 6250 2800 60  0001 C CNN
 	1    6250 2800
@@
 F 0 "L20" H 6850 3038 51  0000 C CNN
 F 1 "YS-SK6812MINI-E" H 6850 3103 16  0000 C CNN
-F 2 "sk6812mini-e:YS-SK6812_backlight" H 6850 3300 60  0001 C CNN
+F 2 "sk6812mini-e:YS-SK6812-MINI-E_backlight" H 6850 3300 60  0001 C CNN
 F 3 "" H 6850 3300 60  0001 C CNN
 	1    6850 3300
@@
 F 0 "L17" H 5050 3038 51  0000 C CNN
 F 1 "YS-SK6812MINI-E" H 5050 3103 16  0000 C CNN
-F 2 "sk6812mini-e:YS-SK6812_backlight" H 5050 3300 60  0001 C CNN
+F 2 "sk6812mini-e:YS-SK6812-MINI-E_backlight" H 5050 3300 60  0001 C CNN
 F 3 "" H 5050 3300 60  0001 C CNN
 	1    5050 3300
@@
 F 0 "L18" H 5650 3038 51  0000 C CNN
 F 1 "YS-SK6812MINI-E" H 5650 3103 16  0000 C CNN
-F 2 "sk6812mini-e:YS-SK6812_backlight" H 5650 3300 60  0001 C CNN
+F 2 "sk6812mini-e:YS-SK6812-MINI-E_backlight" H 5650 3300 60  0001 C CNN
 F 3 "" H 5650 3300 60  0001 C CNN
 	1    5650 3300
@@
 F 0 "L19" H 6250 3038 51  0000 C CNN
 F 1 "YS-SK6812MINI-E" H 6250 3103 16  0000 C CNN
-F 2 "sk6812mini-e:YS-SK6812_backlight" H 6250 3300 60  0001 C CNN
+F 2 "sk6812mini-e:YS-SK6812-MINI-E_backlight" H 6250 3300 60  0001 C CNN
 F 3 "" H 6250 3300 60  0001 C CNN
 	1    6250 3300
@@
 F 0 "L24" H 6850 3538 51  0000 C CNN
 F 1 "YS-SK6812MINI-E" H 6850 3603 16  0000 C CNN
-F 2 "sk6812mini-e:YS-SK6812_backlight" H 6850 3800 60  0001 C CNN
+F 2 "sk6812mini-e:YS-SK6812-MINI-E_backlight" H 6850 3800 60  0001 C CNN
 F 3 "" H 6850 3800 60  0001 C CNN
 	1    6850 3800
@@
 F 0 "L21" H 5050 3538 51  0000 C CNN
 F 1 "YS-SK6812MINI-E" H 5050 3603 16  0000 C CNN
-F 2 "sk6812mini-e:YS-SK6812_backlight" H 5050 3800 60  0001 C CNN
+F 2 "sk6812mini-e:YS-SK6812-MINI-E_backlight" H 5050 3800 60  0001 C CNN
 F 3 "" H 5050 3800 60  0001 C CNN
 	1    5050 3800
@@
 F 0 "L22" H 5650 3538 51  0000 C CNN
 F 1 "YS-SK6812MINI-E" H 5650 3603 16  0000 C CNN
-F 2 "sk6812mini-e:YS-SK6812_backlight" H 5650 3800 60  0001 C CNN
+F 2 "sk6812mini-e:YS-SK6812-MINI-E_backlight" H 5650 3800 60  0001 C CNN
 F 3 "" H 5650 3800 60  0001 C CNN
 	1    5650 3800
@@
 F 0 "L23" H 6250 3538 51  0000 C CNN
 F 1 "YS-SK6812MINI-E" H 6250 3603 16  0000 C CNN
-F 2 "sk6812mini-e:YS-SK6812_backlight" H 6250 3800 60  0001 C CNN
+F 2 "sk6812mini-e:YS-SK6812-MINI-E_backlight" H 6250 3800 60  0001 C CNN
 F 3 "" H 6250 3800 60  0001 C CNN
 	1    6250 3800
@@
 F 0 "L25" H 5050 4038 51  0000 C CNN
 F 1 "YS-SK6812MINI-E" H 5050 4103 16  0000 C CNN
-F 2 "sk6812mini-e:YS-SK6812_backlight" H 5050 4300 60  0001 C CNN
+F 2 "sk6812mini-e:YS-SK6812-MINI-E_backlight" H 5050 4300 60  0001 C CNN
 F 3 "" H 5050 4300 60  0001 C CNN
 	1    5050 4300
@@
 F 0 "L26" H 5650 4038 51  0000 C CNN
 F 1 "YS-SK6812MINI-E" H 5650 4103 16  0000 C CNN
-F 2 "sk6812mini-e:YS-SK6812_backlight" H 5650 4300 60  0001 C CNN
+F 2 "sk6812mini-e:YS-SK6812-MINI-E_backlight" H 5650 4300 60  0001 C CNN
 F 3 "" H 5650 4300 60  0001 C CNN
 	1    5650 4300
@@
 F 0 "L27" H 6250 4038 51  0000 C CNN
 F 1 "YS-SK6812MINI-E" H 6250 4103 16  0000 C CNN
-F 2 "sk6812mini-e:YS-SK6812_backlight" H 6250 4300 60  0001 C CNN
+F 2 "sk6812mini-e:YS-SK6812-MINI-E_backlight" H 6250 4300 60  0001 C CNN
 F 3 "" H 6250 4300 60  0001 C CNN
 	1    6250 4300
@@
 F 0 "L28" H 6850 4038 51  0000 C CNN
 F 1 "YS-SK6812MINI-E" H 6850 4103 16  0000 C CNN
-F 2 "sk6812mini-e:YS-SK6812_backlight" H 6850 4300 60  0001 C CNN
+F 2 "sk6812mini-e:YS-SK6812-MINI-E_backlight" H 6850 4300 60  0001 C CNN
 F 3 "" H 6850 4300 60  0001 C CNN
 	1    6850 4300
@@
 F 0 "L32" H 6850 4538 51  0000 C CNN
 F 1 "YS-SK6812MINI-E" H 6850 4603 16  0000 C CNN
-F 2 "sk6812mini-e:YS-SK6812_backlight" H 6850 4800 60  0001 C CNN
+F 2 "sk6812mini-e:YS-SK6812-MINI-E_backlight" H 6850 4800 60  0001 C CNN
 F 3 "" H 6850 4800 60  0001 C CNN
 	1    6850 4800
@@
 F 0 "L31" H 6250 4538 51  0000 C CNN
 F 1 "YS-SK6812MINI-E" H 6250 4603 16  0000 C CNN
-F 2 "sk6812mini-e:YS-SK6812_backlight" H 6250 4800 60  0001 C CNN
+F 2 "sk6812mini-e:YS-SK6812-MINI-E_backlight" H 6250 4800 60  0001 C CNN
 F 3 "" H 6250 4800 60  0001 C CNN
 	1    6250 4800
@@
 F 0 "L33" H 4350 4538 51  0000 C CNN
 F 1 "YS-SK6812MINI-E" H 4350 4603 16  0000 C CNN
-F 2 "sk6812mini-e:YS-SK6812_backlight" H 4350 4800 60  0001 C CNN
+F 2 "sk6812mini-e:YS-SK6812-MINI-E_backlight" H 4350 4800 60  0001 C CNN
 F 3 "" H 4350 4800 60  0001 C CNN
 	1    4350 4800
@@
 F 0 "L30" H 5650 4538 51  0000 C CNN
 F 1 "YS-SK6812MINI-E" H 5650 4603 16  0000 C CNN
-F 2 "sk6812mini-e:YS-SK6812_backlight" H 5650 4800 60  0001 C CNN
+F 2 "sk6812mini-e:YS-SK6812-MINI-E_backlight" H 5650 4800 60  0001 C CNN
 F 3 "" H 5650 4800 60  0001 C CNN
 	1    5650 4800
@@
 F 0 "L29" H 5050 4538 51  0000 C CNN
 F 1 "YS-SK6812MINI-E" H 5050 4603 16  0000 C CNN
-F 2 "sk6812mini-e:YS-SK6812_backlight" H 5050 4800 60  0001 C CNN
+F 2 "sk6812mini-e:YS-SK6812-MINI-E_backlight" H 5050 4800 60  0001 C CNN
 F 3 "" H 5050 4800 60  0001 C CNN
 	1    5050 4800
@@
 2020-10-29
 Text Notes 10600 7650 0    50   ~ 0
-1.0
+1.1
 $EndSCHEMATC
